Commit message: change IMU color to orange

File: description/imu.xacro (robot description, xacro)
@@ -11,5 +11,5 @@
                 <box size="0.01 0.01 0.01"/>
             </geometry>
-            <material name="red"/>
+            <material name="orange"/>
         </visual>
         <collision>
@@ -20,5 +20,5 @@
     </link>
     <gazebo reference="imu_frame">
-        <material>Gazebo/Red</material>
+        <material>Gazebo/Orange</material>
     </gazebo>
 </robot>
