Commit message: generate 3 robots in empty.world w/ separate namespace

File: description/gazebo_control.xacro (robot description, xacro)
@@ -3,4 +3,9 @@
     <gazebo>
         <plugin name='diff_drive' filename='libgazebo_ros_diff_drive.so'>
+            <ros>
+               <!-- <namespace>robot_1</namespace>
+                <argument>cmd_vel:=cmd_vel</argument>
+                <argument>odom:=odom</argument>   -->
+            </ros>
             <!-- Wheel Information -->
             <left_joint>left_wheel_joint</left_joint>

File: description/robot.urdf.xacro (robot description, xacro)
@@ -1,9 +1,10 @@
 <?xml version="1.0"?>
 <robot xmlns:xacro="http://www.ros.org/wiki/xacro"  name="nsbot">
+    <xacro:arg name="robot_name" default="robot_1"/>
     <!-- include robot core file -->
     <xacro:include filename="robot_core.xacro" />
-    <xacro:include filename="gazebo_control.xacro" />
     <xacro:include filename="imu.xacro" />
     <xacro:include filename="lidar.xacro" />
     <xacro:include filename="camera.xacro" />
+    <!-- <xacro:include filename="gazebo_control.xacro" /> -->
 </robot>

File: description/robot_core.xacro (robot description, xacro)
@@ -1,4 +1,5 @@
 <?xml version="1.0"?>
-<robot xmlns:xacro="http://www.ros.org/wiki/xacro" >
+<robot xmlns:xacro="http://www.ros.org/wiki/xacro" name="nsbot" >
+    <xacro:arg name="robot_name" default=""/>
     <xacro:include filename="inertial_macros.xacro"/>
     <material name="white">
@@ -38,5 +39,5 @@
         </collision>
         <xacro:inertial_box mass="0.5" x="0.3" y="0.3" z="0.15">
-            <origin xyz="0.15 0 0.075" rpy="0 0 0"/>
+            <origin xyz="0.15 0 -0.075" rpy="0 0 0"/>
         </xacro:inertial_box>
     </link>
@@ -123,3 +124,79 @@
         <mu2 value="0.001"/>
     </gazebo>
+<!-- Define LIDAR -->
+    <joint name="laser_joint" type="fixed">
+        <parent link="chassis"/>
+        <child link="laser_link"/>
+        <origin xyz="0.1 0 0.175" rpy="0 0 0"/>
+    </joint>
+    <link name="laser_link">
+        <visual>
+            <geometry>
+                <cylinder radius="0.05" length="0.04"/>
+            </geometry>
+            <material name="red"/>
+        </visual>
+        <collision>
+            <geometry>
+                <cylinder radius="0.05" length="0.04"/>
+            </geometry>
+        </collision>
+        <xacro:inertial_cylinder mass="0.1" length="0.04" radius="0.05">
+            <origin xyz="0 0 0" rpy="0 0 0"/>
+        </xacro:inertial_cylinder>
+    </link>
+    <material name="red">
+        <color rgba="1 0 0 1"/>
+    </material>
+    <gazebo reference="laser_link">
+        <material>Gazebo/Red</material>
+        <sensor name="laser" type="ray">
+            <pose> 0 0 0 0 0 0 </pose>
+            <visualize>true</visualize>
+            <update_rate>10</update_rate>
+            <ray>
+                <scan>
+                    <horizontal>
+                        <samples>360</samples>
+                        <min_angle>-3.14</min_angle>
+                        <max_angle>3.14</max_angle>
+                    </horizontal>
+                </scan>
+                <range>
+                    <min>0.3</min>
+                    <max>12</max>
+                </range>
+            </ray>
+            <plugin name="laser_controller" filename="libgazebo_ros_ray_sensor.so">
+                <ros>
+                    <argument>~/out:=scan</argument>
+                </ros>
+                <output_type>sensor_msgs/LaserScan</output_type>
+                <frame_name>laser_link</frame_name>
+            </plugin>
+        </sensor>
+    </gazebo>
+    <gazebo>
+        <plugin name='diff_drive' filename='libgazebo_ros_diff_drive.so'>
+            <ros>
+           <!-- <namespace>/</namespace>
+                <argument>cmd_vel:=cmd_vel</argument>
+                <argument>odom:=odom</argument>   -->
+            </ros>
+            <!-- Wheel Information -->
+            <left_joint>left_wheel_joint</left_joint>
+            <right_joint>right_wheel_joint</right_joint>
+            <wheel_separation>0.35</wheel_separation>
+            <wheel_diameter>0.1</wheel_diameter>
+            <!-- Limits -->
+            <max_wheel_torque>200</max_wheel_torque>
+            <max_wheel_acceleration>10.0</max_wheel_acceleration>
+            <!-- Output -->
+            <odometry_frame>$(arg robot_name)/odom</odometry_frame>
+            <robot_base_frame>$(arg robot_name)/base_link</robot_base_frame>
+            <publish_odom>true</publish_odom>
+            <publish_odom_tf>true</publish_odom_tf>
+            <publish_wheel_tf>true</publish_wheel_tf>
+        </plugin>
+    </gazebo>
 </robot>

Commit message: v1.0 working version

File: description/gazebo_control.xacro (robot description, xacro)
@@ -4,7 +4,5 @@
         <plugin name='diff_drive' filename='libgazebo_ros_diff_drive.so'>
             <ros>
-               <!-- <namespace>robot_1</namespace>
-                <argument>cmd_vel:=cmd_vel</argument>
-                <argument>odom:=odom</argument>   -->
+                <!-- <argument>/tf:=/$(arg robot_name)/tf</argument>  -->
             </ros>
             <!-- Wheel Information -->
@@ -17,9 +15,13 @@
             <max_wheel_acceleration>10.0</max_wheel_acceleration>
             <!-- Output -->
-            <odometry_frame>odom</odometry_frame>
-            <robot_base_frame>base_link</robot_base_frame>
-            <publish_odom>true</publish_odom>
-            <publish_odom_tf>true</publish_odom_tf>
-            <publish_wheel_tf>true</publish_wheel_tf>
+            <odometry_frame>$(arg robot_name)/odom</odometry_frame>
+            <robot_base_frame>$(arg robot_name)/base_link</robot_base_frame>
+            <odometrySource>0</odometrySource>
+            <publish_odom>True</publish_odom>
+            <publish_odom_tf>True</publish_odom_tf>
+            <publish_wheel_tf>False</publish_wheel_tf>
+            <publishWheelJointState>True</publishWheelJointState>
+            <!--
+            -->
         </plugin>
     </gazebo>

File: description/imu.xacro (robot description, xacro)
@@ -21,4 +21,23 @@
     <gazebo reference="imu_frame">
         <material>Gazebo/Orange</material>
+        <sensor name="imu" type="imu">
+            <always_on>true</always_on>
+            <update_rate>100</update_rate>
+            <visualize>true</visualize>
+            <topic>__default_topic__</topic>
+            <plugin name="imu" filename="libgazebo_ros_imu_sensor.so">
+                 <ros>
+                     <argument>~/out:=~/data</argument>
+                 </ros>
+                 <topicName>imu_frame</topicName>
+                 <bodyName>imu_frame</bodyName>
+                 <gaussianNoise>0.0</gaussianNoise>
+                 <xyzOffset>0 0 0</xyzOffset>
+                 <rpyOffset>0 0 0</rpyOffset>
+                 <frameName>imu_frame</frameName>
+                 <initialOrientationAsReference>false</initialOrientationAsReference>
+            </plugin>
+            <pose>0 0 0 0 0 0</pose>
+        </sensor>
     </gazebo>
 </robot>

File: description/robot.urdf.xacro (robot description, xacro)
@@ -1,5 +1,5 @@
 <?xml version="1.0"?>
 <robot xmlns:xacro="http://www.ros.org/wiki/xacro"  name="nsbot">
-    <xacro:arg name="robot_name" default="robot_1"/>
+    <xacro:arg name="robot_name" default=""/>
     <!-- include robot core file -->
     <xacro:include filename="robot_core.xacro" />
@@ -7,4 +7,4 @@
     <xacro:include filename="lidar.xacro" />
     <xacro:include filename="camera.xacro" />
-    <!-- <xacro:include filename="gazebo_control.xacro" /> -->
+    <xacro:include filename="gazebo_control.xacro" />
 </robot>

File: description/robot_core.xacro (robot description, xacro)
@@ -1,5 +1,4 @@
 <?xml version="1.0"?>
 <robot xmlns:xacro="http://www.ros.org/wiki/xacro" name="nsbot" >
-    <xacro:arg name="robot_name" default=""/>
     <xacro:include filename="inertial_macros.xacro"/>
     <material name="white">
@@ -124,79 +123,3 @@
         <mu2 value="0.001"/>
     </gazebo>
-<!-- Define LIDAR -->
-    <joint name="laser_joint" type="fixed">
-        <parent link="chassis"/>
-        <child link="laser_link"/>
-        <origin xyz="0.1 0 0.175" rpy="0 0 0"/>
-    </joint>
-    <link name="laser_link">
-        <visual>
-            <geometry>
-                <cylinder radius="0.05" length="0.04"/>
-            </geometry>
-            <material name="red"/>
-        </visual>
-        <collision>
-            <geometry>
-                <cylinder radius="0.05" length="0.04"/>
-            </geometry>
-        </collision>
-        <xacro:inertial_cylinder mass="0.1" length="0.04" radius="0.05">
-            <origin xyz="0 0 0" rpy="0 0 0"/>
-        </xacro:inertial_cylinder>
-    </link>
-    <material name="red">
-        <color rgba="1 0 0 1"/>
-    </material>
-    <gazebo reference="laser_link">
-        <material>Gazebo/Red</material>
-        <sensor name="laser" type="ray">
-            <pose> 0 0 0 0 0 0 </pose>
-            <visualize>true</visualize>
-            <update_rate>10</update_rate>
-            <ray>
-                <scan>
-                    <horizontal>
-                        <samples>360</samples>
-                        <min_angle>-3.14</min_angle>
-                        <max_angle>3.14</max_angle>
-                    </horizontal>
-                </scan>
-                <range>
-                    <min>0.3</min>
-                    <max>12</max>
-                </range>
-            </ray>
-            <plugin name="laser_controller" filename="libgazebo_ros_ray_sensor.so">
-                <ros>
-                    <argument>~/out:=scan</argument>
-                </ros>
-                <output_type>sensor_msgs/LaserScan</output_type>
-                <frame_name>laser_link</frame_name>
-            </plugin>
-        </sensor>
-    </gazebo>
-    <gazebo>
-        <plugin name='diff_drive' filename='libgazebo_ros_diff_drive.so'>
-            <ros>
-           <!-- <namespace>/</namespace>
-                <argument>cmd_vel:=cmd_vel</argument>
-                <argument>odom:=odom</argument>   -->
-            </ros>
-            <!-- Wheel Information -->
-            <left_joint>left_wheel_joint</left_joint>
-            <right_joint>right_wheel_joint</right_joint>
-            <wheel_separation>0.35</wheel_separation>
-            <wheel_diameter>0.1</wheel_diameter>
-            <!-- Limits -->
-            <max_wheel_torque>200</max_wheel_torque>
-            <max_wheel_acceleration>10.0</max_wheel_acceleration>
-            <!-- Output -->
-            <odometry_frame>$(arg robot_name)/odom</odometry_frame>
-            <robot_base_frame>$(arg robot_name)/base_link</robot_base_frame>
-            <publish_odom>true</publish_odom>
-            <publish_odom_tf>true</publish_odom_tf>
-            <publish_wheel_tf>true</publish_wheel_tf>
-        </plugin>
-    </gazebo>
 </robot>
