Commit message: v2.0 fixing no scan points problem of liadar sensors

File: description/lidar.xacro (robot description, xacro)
@@ -29,10 +29,10 @@
         <sensor name="laser" type="ray">
             <pose> 0 0 0 0 0 0 </pose>
-            <visualize>true</visualize>
-            <update_rate>10</update_rate>
+            <visualize>false</visualize>
+            <update_rate>5</update_rate>
             <ray>
                 <scan>
                     <horizontal>
-                        <samples>360</samples>
+                        <samples>120</samples>
                         <min_angle>-3.14</min_angle>
                         <max_angle>3.14</max_angle>
@@ -49,5 +49,5 @@
                 </ros>
                 <output_type>sensor_msgs/LaserScan</output_type>
-                <frame_name>laser_link</frame_name>
+                <frame_name>$(arg robot_name)/laser_link</frame_name>
             </plugin>
         </sensor>

File: description/robot_core.xacro (robot description, xacro)
@@ -38,5 +38,5 @@
         </collision>
         <xacro:inertial_box mass="0.5" x="0.3" y="0.3" z="0.15">
-            <origin xyz="0.15 0 -0.075" rpy="0 0 0"/>
+            <origin xyz="0.15 0 0.075" rpy="0 0 0"/>
         </xacro:inertial_box>
     </link>
